File: PLACA DRIVER RSENSE 10A.kicad_sch (KiCad schematic)
At the start: 27 parts, among them J1 AVR_SPI_PRG_6PTH, U1 Tiny45-20-SMT, Y1 8Mhz

Commit message: Schematic atualizado automaticamente - Componentes corrigidos
Alteracoes automaticas realizadas:
- Indutor: NR8040T100M -> SRP1265A-100M 10uH 12A
- C3: 47uF 63V -> 100uF 63V
- C4: 4.7uF 80V -> 10uF 100V
- D1: Footprint SMA -> SMC

Arquivos incluidos:
- PLACA DRIVER RSENSE 10A.kicad_sch (ATUALIZADO)
- PLACA DRIVER RSENSE 10A.kicad_pcb
- atualizar_projeto.py (script de automacao)
- ALTERACOES_AUTOMATICAS.txt (relatorio)
Parts:
- C3: value 47uF 63V -> 100uF 63V
- C4: value 4.7uF 80V -> 10uF 100V
- D1: footprint Placa_Driver_Alpha_2026:SMA -> Placa_Driver_Alpha_2026:SMC
- U$3: value 10uH -> SRP1265A-100M 10uH 12A
Changed lines of the file:
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@@
 			)
 		)
-		(property "Value" "10uH"
+		(property "Value" "SRP1265A-100M 10uH 12A"
 			(at 215.9 35.56 0)
 			(effects
@@
 			)
 		)
-		(property "Value" "4.7uF 80V"
+		(property "Value" "10uF 100V"
 			(at 103.124 58.039 0)
 			(effects
@@
 			)
 		)
-		(property "Value" "47uF 63V"
+		(property "Value" "100uF 63V"
 			(at 84.836 57.531 0)
 			(effects
@@
 			)
 		)
-		(property "Footprint" "Placa_Driver_Alpha_2026:SMA"
+		(property "Footprint" "Placa_Driver_Alpha_2026:SMC"
 			(at 200.66 60.96 0)
 			(effects
