File: PLACA DRIVER RSENSE 10A.kicad_pcb (KiCad board)
At the start: 4 copper layers, 29.4 x 26 mm, 27 parts, among them J1 AVR_SPI_PRG_6PTH, U1 Tiny45-20-SMT, Y1 8Mhz

Commit message: PCB atualizado com componentes corrigidos - Indutor 12A, C3 100uF, C4 10uF
Parts:
- C3: value 47uF 63V -> 100uF 63V
- C4: value 4.7uF 80V -> 10uF 100V
- U$3: value 10uH -> SRP1265A-100M 10uH 12A
Changed lines of the file:
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@@
 			)
 		)
-		(property "Value" "4.7uF 80V"
+		(property "Value" "10uF 100V"
 			(at -1.905 3.175 90)
 			(unlocked yes)
@@
 			)
 		)
-		(property "Value" "10uH"
+		(property "Value" "SRP1265A-100M 10uH 12A"
 			(at 1.6 3.7 90)
 			(unlocked yes)
@@
 		(at 139.7761 108.3536 90)
 		(property "Reference" "SJ1"
-			(at -0.908 1.27 -90)
+			(at -0.908 1.27 270)
 			(unlocked yes)
 			(layer "B.SilkS")
@@
 		)
 		(property "Value" "JUMPER-PAD-2-NO"
-			(at -0.908 -1.651 -90)
+			(at -0.908 -1.651 270)
 			(unlocked yes)
 			(layer "B.Fab")
@@
 		)
 		(property "Datasheet" ""
-			(at 0 0 -90)
+			(at 0 0 270)
 			(layer "B.Fab")
 			(hide yes)
@@
 		)
 		(property "Description" ""
-			(at 0 0 -90)
+			(at 0 0 270)
 			(layer "B.Fab")
 			(hide yes)
@@
 		(descr "CAPACITOR")
 		(property "Reference" "C8"
-			(at -0.935 0.635 -90)
+			(at -0.935 0.635 270)
 			(unlocked yes)
 			(layer "B.SilkS")
@@
 		)
 		(property "Value" "0.1uF"
-			(at -0.935 -1.105 -90)
+			(at -0.935 -1.105 270)
 			(unlocked yes)
 			(layer "B.Fab")
@@
 		)
 		(property "Datasheet" ""
-			(at 0 0 -90)
+			(at 0 0 270)
 			(layer "B.Fab")
 			(hide yes)
@@
 		)
 		(property "Description" ""
-			(at 0 0 -90)
+			(at 0 0 270)
 			(layer "B.Fab")
 			(hide yes)
@@
 		(descr "CAPACITOR")
 		(property "Reference" "C6"
-			(at -0.635 0.635 -90)
+			(at -0.635 0.635 270)
 			(unlocked yes)
 			(layer "B.SilkS")
@@
 		)
 		(property "Value" "10uF"
-			(at -0.635 -1.27 -90)
+			(at -0.635 -1.27 270)
 			(unlocked yes)
 			(layer "B.Fab")
@@
 		)
 		(property "Datasheet" ""
-			(at 0 0 -90)
+			(at 0 0 270)
 			(layer "B.Fab")
 			(hide yes)
@@
 		)
 		(property "Description" ""
-			(at 0 0 -90)
+			(at 0 0 270)
 			(layer "B.Fab")
 			(hide yes)
@@
 		(descr "RESISTOR")
 		(property "Reference" "R9"
-			(at -0.889 0.635 -90)
+			(at -0.889 0.635 270)
 			(unlocked yes)
 			(layer "B.SilkS")
@@
 		)
 		(property "Value" "3.3K 1%"
-			(at -0.889 -1.016 -90)
+			(at -0.889 -1.016 270)
 			(unlocked yes)
 			(layer "B.Fab")
@@
 		)
 		(property "Datasheet" ""
-			(at 0 0 -90)
+			(at 0 0 270)
 			(layer "B.Fab")
 			(hide yes)
@@
 		)
 		(property "Description" ""
-			(at 0 0 -90)
+			(at 0 0 270)
 			(layer "B.Fab")
 			(hide yes)
@@
 		(at 141.544428 99.056588 -90)
 		(property "Reference" "C3"
-			(at -0.762 1.651 -90)
+			(at -0.762 1.651 270)
 			(unlocked yes)
 			(layer "B.SilkS")
@@
 			)
 		)
-		(property "Value" "47uF 63V"
-			(at -1.905 -4.318 -90)
+		(property "Value" "100uF 63V"
+			(at -1.905 -4.318 270)
 			(unlocked yes)
 			(layer "B.Fab")
@@
 		(descr "RESISTOR")
 		(property "Reference" "R4"
-			(at -0.889 0.635 -90)
+			(at -0.889 0.635 270)
 			(unlocked yes)
 			(layer "B.SilkS")
@@
 		)
 		(property "Value" "10K"
-			(at -0.889 -1.016 -90)
+			(at -0.889 -1.016 270)
 			(unlocked yes)
 			(layer "B.Fab")
@@
 		)
 		(property "Datasheet" ""
-			(at 0 0 -90)
+			(at 0 0 270)
 			(layer "B.Fab")
 			(hide yes)
@@
 		)
 		(property "Description" ""
-			(at 0 0 -90)
+			(at 0 0 270)
 			(layer "B.Fab")
 			(hide yes)
